File: externalTemperature/externalTempProbe.sch (KiCad schematic (older format))
At the start: 5 parts

Commit message: ran rescue
Parts:
- C? (x3): symbol C -> C-RESCUE-externalTempProbe
Changed lines of the file:
@@
 EESchema Schematic File Version 2
+LIBS:externalTempProbe-rescue
 LIBS:power
 LIBS:device
@@
 $EndComp
 $Comp
-L GNDA #PWR?
+L GNDA-RESCUE-externalTempProbe #PWR?
 U 1 1 559476F7
 P 5100 3900
@@
 $EndComp
 $Comp
-L C C?
+L C-RESCUE-externalTempProbe C?
 U 1 1 5594C942
 P 4700 3900
@@
 Connection ~ 4700 3700
 $Comp
-L GNDA #PWR?
+L GNDA-RESCUE-externalTempProbe #PWR?
 U 1 1 55959F33
 P 4700 4100
@@
 $EndComp
 $Comp
-L GNDA #PWR?
+L GNDA-RESCUE-externalTempProbe #PWR?
 U 1 1 5594B819
 P 7100 3900
@@
 SCL
 $Comp
-L C C?
+L C-RESCUE-externalTempProbe C?
 U 1 1 55961C1D
 P 4450 3900
@@
 $EndComp
 $Comp
-L C C?
+L C-RESCUE-externalTempProbe C?
 U 1 1 55961C58
 P 4200 3900
@@
 Connection ~ 4450 3700
 $Comp
-L GNDA #PWR?
+L GNDA-RESCUE-externalTempProbe #PWR?
 U 1 1 55961D3C
 P 4200 4100
@@
 $EndComp
 $Comp
-L GNDA #PWR?
+L GNDA-RESCUE-externalTempProbe #PWR?
 U 1 1 55961D55
 P 4450 4100
@@
 $EndComp
 $Comp
-L GNDA #PWR?
+L GNDA-RESCUE-externalTempProbe #PWR?
 U 1 1 55961F67
 P 6150 3700
