File: power.sch (KiCad schematic (older format))
At the start: 31 parts

Commit message: did more work
Parts:
- added D?: D_Schottky, symbol D_Schottky
- added R? (x2): 100K, symbol R
- R?: value 100K -> 10K
Connections:
- net labels added: BUTTON
- wire segments 64 -> 70
Changed lines of the file:
@@
 $EndComp
 $Comp
-L GND-RESCUE-cansatBrain #PWR038
+L GND-RESCUE-cansatBrain #PWR037
 U 1 1 5594EE74
 P 1900 1750
-F 0 "#PWR038" H 1900 1750 30  0001 C CNN
+F 0 "#PWR037" H 1900 1750 30  0001 C CNN
 F 1 "GND" H 1900 1680 30  0001 C CNN
 F 2 "" H 1900 1750 60  0000 C CNN
@@
 $EndComp
 $Comp
-L GND-RESCUE-cansatBrain #PWR039
+L GND-RESCUE-cansatBrain #PWR038
 U 1 1 5594EE7A
 P 3150 1750
-F 0 "#PWR039" H 3150 1750 30  0001 C CNN
+F 0 "#PWR038" H 3150 1750 30  0001 C CNN
 F 1 "GND" H 3150 1680 30  0001 C CNN
 F 2 "" H 3150 1750 60  0000 C CNN
@@
 $EndComp
 $Comp
-L GND-RESCUE-cansatBrain #PWR040
+L GND-RESCUE-cansatBrain #PWR039
 U 1 1 5594EE80
 P 1300 1750
-F 0 "#PWR040" H 1300 1750 30  0001 C CNN
+F 0 "#PWR039" H 1300 1750 30  0001 C CNN
 F 1 "GND" H 1300 1680 30  0001 C CNN
 F 2 "" H 1300 1750 60  0000 C CNN
@@
 $EndComp
 $Comp
-L GND-RESCUE-cansatBrain #PWR041
+L GND-RESCUE-cansatBrain #PWR040
 U 1 1 5594EE86
 P 1000 1650
-F 0 "#PWR041" H 1000 1650 30  0001 C CNN
+F 0 "#PWR040" H 1000 1650 30  0001 C CNN
 F 1 "GND" H 1000 1580 30  0001 C CNN
 F 2 "" H 1000 1650 60  0000 C CNN
@@
 $EndComp
 $Comp
-L GND-RESCUE-cansatBrain #PWR042
+L GND-RESCUE-cansatBrain #PWR041
 U 1 1 5594EE8C
 P 3550 1650
-F 0 "#PWR042" H 3550 1650 30  0001 C CNN
+F 0 "#PWR041" H 3550 1650 30  0001 C CNN
 F 1 "GND" H 3550 1580 30  0001 C CNN
 F 2 "" H 3550 1650 60  0000 C CNN
@@
 $EndComp
 $Comp
-L VCC #PWR043
+L VCC #PWR042
 U 1 1 5594EE92
 P 3550 1250
-F 0 "#PWR043" H 3550 1350 30  0001 C CNN
+F 0 "#PWR042" H 3550 1350 30  0001 C CNN
 F 1 "VCC" H 3550 1350 30  0000 C CNN
 F 2 "" H 3550 1250 60  0000 C CNN
@@
 $EndComp
 $Comp
-L GND-RESCUE-cansatBrain #PWR044
+L GND-RESCUE-cansatBrain #PWR043
 U 1 1 5594EE9F
 P 3800 1650
-F 0 "#PWR044" H 3800 1650 30  0001 C CNN
+F 0 "#PWR043" H 3800 1650 30  0001 C CNN
 F 1 "GND" H 3800 1580 30  0001 C CNN
 F 2 "" H 3800 1650 60  0000 C CNN
@@
 P 10150 2900
 F 0 "R?" V 10230 2900 40  0000 C CNN
-F 1 "100K" V 10157 2901 40  0000 C CNN
+F 1 "10K" V 10157 2901 40  0000 C CNN
 F 2 "" V 10080 2900 30  0000 C CNN
 F 3 "" H 10150 2900 30  0000 C CNN
@@
 $EndComp
 $Comp
-L VCCA #PWR046
+L VCCA #PWR044
 U 1 1 55952BE9
 P 9800 1450
-F 0 "#PWR046" H 9800 1550 30  0001 C CNN
+F 0 "#PWR044" H 9800 1550 30  0001 C CNN
 F 1 "VCCA" H 9800 1550 30  0000 C CNN
 F 2 "" H 9800 1450 60  0000 C CNN
@@
 $EndComp
 $Comp
-L VCC #PWR047
+L VCC #PWR045
 U 1 1 55952BF6
 P 9200 1450
-F 0 "#PWR047" H 9200 1550 30  0001 C CNN
+F 0 "#PWR045" H 9200 1550 30  0001 C CNN
 F 1 "VCC" H 9200 1550 30  0000 C CNN
 F 2 "" H 9200 1450 60  0000 C CNN
@@
 $EndComp
 $Comp
-L GNDA-RESCUE-cansatBrain #PWR048
+L GNDA-RESCUE-cansatBrain #PWR046
 U 1 1 55952BFE
 P 9800 1800
-F 0 "#PWR048" H 9800 1800 40  0001 C CNN
+F 0 "#PWR046" H 9800 1800 40  0001 C CNN
 F 1 "GNDA" H 9800 1730 40  0000 C CNN
 F 2 "" H 9800 1800 60  0000 C CNN
@@
 $EndComp
 $Comp
-L GND-RESCUE-cansatBrain #PWR049
+L GND-RESCUE-cansatBrain #PWR047
 U 1 1 55952C04
 P 9200 1800
-F 0 "#PWR049" H 9200 1800 30  0001 C CNN
+F 0 "#PWR047" H 9200 1800 30  0001 C CNN
 F 1 "GND" H 9200 1730 30  0001 C CNN
 F 2 "" H 9200 1800 60  0000 C CNN
@@
 Text HLabel 1900 1450 0    60   Input ~ 0
 REG_EN
-Text HLabel 8800 2900 0    60   Input ~ 0
+Text HLabel 8150 2150 0    60   Input ~ 0
 REG_EN
 $Comp
@@
 $EndComp
 $Comp
-L GND-RESCUE-cansatBrain #PWR050
+L GND-RESCUE-cansatBrain #PWR048
 U 1 1 55955FDC
 P 9250 6050
-F 0 "#PWR050" H 9250 6050 30  0001 C CNN
+F 0 "#PWR048" H 9250 6050 30  0001 C CNN
 F 1 "GND" H 9250 5980 30  0001 C CNN
 F 2 "" H 9250 6050 60  0000 C CNN
@@
 $EndComp
 $Comp
-L GND #PWR051
+L GND #PWR049
 U 1 1 56DF83C7
 P 1050 4750
-F 0 "#PWR051" H 1050 4500 50  0001 C CNN
+F 0 "#PWR049" H 1050 4500 50  0001 C CNN
 F 1 "GND" H 1050 4600 50  0000 C CNN
 F 2 "" H 1050 4750 50  0000 C CNN
@@
 $EndComp
 $Comp
-L GND #PWR052
+L GND #PWR050
 U 1 1 56DFA497
 P 1900 3550
-F 0 "#PWR052" H 1900 3300 50  0001 C CNN
+F 0 "#PWR050" H 1900 3300 50  0001 C CNN
 F 1 "GND" H 1900 3400 50  0000 C CNN
 F 2 "" H 1900 3550 50  0000 C CNN
@@
 Disconnect battery when \nUSB power is available
 $Comp
-L +5V #PWR053
+L +5V #PWR051
 U 1 1 56DFC2FC
 P 6900 2800
-F 0 "#PWR053" H 6900 2650 50  0001 C CNN
+F 0 "#PWR051" H 6900 2650 50  0001 C CNN
 F 1 "+5V" H 6900 2940 50  0000 C CNN
 F 2 "" H 6900 2800 50  0000 C CNN
@@
 $EndComp
 $Comp
-L GND #PWR054
+L GND #PWR052
 U 1 1 56DFFA3D
 P 5400 3150
-F 0 "#PWR054" H 5400 2900 50  0001 C CNN
+F 0 "#PWR052" H 5400 2900 50  0001 C CNN
 F 1 "GND" H 5400 3000 50  0000 C CNN
 F 2 "" H 5400 3150 50  0000 C CNN
@@
 $EndComp
 $Comp
-L GND #PWR055
+L GND #PWR053
 U 1 1 56E0020E
 P 5300 3800
-F 0 "#PWR055" H 5300 3550 50  0001 C CNN
+F 0 "#PWR053" H 5300 3550 50  0001 C CNN
 F 1 "GND" H 5300 3650 50  0000 C CNN
 F 2 "" H 5300 3800 50  0000 C CNN
@@
 $EndComp
 $Comp
-L GND #PWR056
+L GND #PWR054
 U 1 1 56E00B62
 P 6000 4000
-F 0 "#PWR056" H 6000 3750 50  0001 C CNN
+F 0 "#PWR054" H 6000 3750 50  0001 C CNN
 F 1 "GND" H 6000 3850 50  0000 C CNN
 F 2 "" H 6000 4000 50  0000 C CNN
@@
 $EndComp
 $Comp
-L GND #PWR057
+L GND #PWR055
 U 1 1 56E025B4
 P 7250 3200
-F 0 "#PWR057" H 7250 2950 50  0001 C CNN
+F 0 "#PWR055" H 7250 2950 50  0001 C CNN
 F 1 "GND" H 7250 3050 50  0000 C CNN
 F 2 "" H 7250 3200 50  0000 C CNN
@@
 $EndComp
 $Comp
-L GND #PWR058
+L GND #PWR056
 U 1 1 56E05829
 P 4250 3150
-F 0 "#PWR058" H 4250 2900 50  0001 C CNN
+F 0 "#PWR056" H 4250 2900 50  0001 C CNN
 F 1 "GND" H 4250 3000 50  0000 C CNN
 F 2 "" H 4250 3150 50  0000 C CNN
@@
 NoConn ~ 6600 3350
 $Comp
-L +5V #PWR?
+L +5V #PWR057
 U 1 1 56E09B9F
 P 1200 1100
-F 0 "#PWR?" H 1200 950 50  0001 C CNN
+F 0 "#PWR057" H 1200 950 50  0001 C CNN
 F 1 "+5V" H 1200 1240 50  0000 C CNN
 F 2 "" H 1200 1100 50  0000 C CNN
@@
 $EndComp
 $Comp
-L GND #PWR?
+L GND #PWR058
 U 1 1 56DF79F7
 P 1000 6750
-F 0 "#PWR?" H 1000 6500 50  0001 C CNN
+F 0 "#PWR058" H 1000 6500 50  0001 C CNN
 F 1 "GND" H 1000 6600 50  0000 C CNN
 F 2 "" H 1000 6750 50  0000 C CNN
@@
 	1000 5700 1000 5550
 $Comp
-L +5V #PWR?
+L +5V #PWR059
 U 1 1 56DFA3E3
 P 1000 5550
-F 0 "#PWR?" H 1000 5400 50  0001 C CNN
+F 0 "#PWR059" H 1000 5400 50  0001 C CNN
 F 1 "+5V" H 1000 5690 50  0000 C CNN
 F 2 "" H 1000 5550 50  0000 C CNN
@@
 $EndComp
 $Comp
-L GND #PWR?
+L GND #PWR060
 U 1 1 56DFB509
 P 1750 6300
-F 0 "#PWR?" H 1750 6050 50  0001 C CNN
+F 0 "#PWR060" H 1750 6050 50  0001 C CNN
 F 1 "GND" H 1750 6150 50  0000 C CNN
 F 2 "" H 1750 6300 50  0000 C CNN
@@
 $EndComp
 Wire Wire Line
-	9250 2900 8800 2900
-Wire Wire Line
-	9100 3000 9100 2900
+	8500 2900 9250 2900
+Wire Wire Line
+	9100 2900 9100 3000
 Connection ~ 9100 2900
 Wire Wire Line
 	9100 3400 9100 3550
 $Comp
-L GND #PWR?
+L GND #PWR061
 U 1 1 56E0CBC0
 P 9100 3550
-F 0 "#PWR?" H 9100 3300 50  0001 C CNN
+F 0 "#PWR061" H 9100 3300 50  0001 C CNN
 F 1 "GND" H 9100 3400 50  0000 C CNN
 F 2 "" H 9100 3550 50  0000 C CNN
@@
 	1    0    0    -1
 $EndComp
+Text HLabel 8500 2900 0    60   Output ~ 0
+BUTTON
+$Comp
+L R R?
+U 1 1 56E03E18
+P 8800 3200
+F 0 "R?" V 8880 3200 50  0000 C CNN
+F 1 "100K" V 8800 3200 50  0000 C CNN
+F 2 "" V 8730 3200 50  0000 C CNN
+F 3 "" H 8800 3200 50  0000 C CNN
+	1    8800 3200
+	1    0    0    -1
+$EndComp
+Wire Wire Line
+	8800 3050 8800 2900
+Connection ~ 8800 2900
+Wire Wire Line
+	8800 3350 8800 3550
+$Comp
+L GND #PWR062
+U 1 1 56E05399
+P 8800 3550
+F 0 "#PWR062" H 8800 3300 50  0001 C CNN
+F 1 "GND" H 8800 3400 50  0000 C CNN
+F 2 "" H 8800 3550 50  0000 C CNN
+F 3 "" H 8800 3550 50  0000 C CNN
+	1    8800 3550
+	1    0    0    -1
+$EndComp
+$Comp
+L D_Schottky D?
+U 1 1 56E062ED
+P 8750 2150
+F 0 "D?" H 8750 2250 50  0000 C CNN
+F 1 "D_Schottky" H 8750 2050 50  0000 C CNN
+F 2 "" H 8750 2150 50  0000 C CNN
+F 3 "" H 8750 2150 50  0000 C CNN
+	1    8750 2150
+	1    0    0    -1
+$EndComp
+Connection ~ 9000 2900
+Wire Wire Line
+	8600 2150 8150 2150
+Wire Wire Line
+	8900 2150 9000 2150
+Wire Wire Line
+	9000 2150 9000 2900
+$Comp
+L R R?
+U 1 1 56E081E9
+P 8300 2350
+F 0 "R?" V 8380 2350 50  0000 C CNN
+F 1 "100K" V 8300 2350 50  0000 C CNN
+F 2 "" V 8230 2350 50  0000 C CNN
+F 3 "" H 8300 2350 50  0000 C CNN
+	1    8300 2350
+	1    0    0    -1
+$EndComp
+$Comp
+L GND #PWR063
+U 1 1 56E082AF
+P 8300 2500
+F 0 "#PWR063" H 8300 2250 50  0001 C CNN
+F 1 "GND" H 8300 2350 50  0000 C CNN
+F 2 "" H 8300 2500 50  0000 C CNN
+F 3 "" H 8300 2500 50  0000 C CNN
+	1    8300 2500
+	1    0    0    -1
+$EndComp
+Wire Wire Line
+	8300 2200 8300 2150
+Connection ~ 8300 2150
 $EndSCHEMATC

Commit message: more stuff
Parts:
- removed BT?: BATTERY, symbol BATTERY
- gave numbers to parts that had none: 33
Connections:
- wire segments 70 -> 73
- no-connect marks 1 -> 3
Other:
- note added: "2 CR2 lithium\ncells in series"
- note removed: "CR2 lithium cell"

Commit message: footprints
Parts:
- BT1, BT2: footprint (none) -> Pin_Headers:Pin_Header_Straight_1x02
- C15, C16, C17, C18, C19, C20, C21, C22, C23, C24: footprint (none) -> Capacitors_SMD:C_0402
- D1, D2, D3: footprint (none) -> Diodes_SMD:MELF-RM10_Universal_Handsoldering
- L1, L2: footprint (none) -> Inductors:IND_BOURNS_SRP1238A
- L3, L4: footprint (none) -> Choke_Axial_ThroughHole:Choke_Horizontal_RM10mm
- Q4, Q5, Q6: footprint (none) -> TO_SOT_Packages_SMD:SOT-23_Handsoldering
- R14, R15, R16, R17, R18, R19, R20, R21: footprint (none) -> Resistors_SMD:R_0402
- SW1: footprint (none) -> Buttons_Switches_ThroughHole:SW_TH_Tactile_Omron_B3F-10xx
- U8, U9: footprint (none) -> Housings_SSOP:MSOP-10-1EP_3x3mm_Pitch0.5mm
Changed lines of the file:
@@
 F 0 "U8" H 2200 1800 60  0000 C CNN
 F 1 "TPS63031" H 2350 1000 60  0000 C CNN
-F 2 "" H 2650 1000 60  0000 C CNN
+F 2 "Housings_SSOP:MSOP-10-1EP_3x3mm_Pitch0.5mm" H 2650 1000 60  0001 C CNN
 F 3 "" H 2650 1000 60  0000 C CNN
 	1    2500 1400
@@
 F 0 "L1" V 2450 850 40  0000 C CNN
 F 1 "1.5 uH" V 2600 850 40  0000 C CNN
-F 2 "" H 2500 850 60  0000 C CNN
+F 2 "Inductors:IND_BOURNS_SRP1238A" H 2500 850 60  0001 C CNN
 F 3 "" H 2500 850 60  0000 C CNN
 	1    2500 850
@@
 F 0 "C15" H 1000 1550 40  0000 L CNN
 F 1 "10 uF" H 1006 1365 40  0000 L CNN
-F 2 "" H 1038 1300 30  0000 C CNN
+F 2 "Capacitors_SMD:C_0402" H 1038 1300 30  0001 C CNN
 F 3 "" H 1000 1450 60  0000 C CNN
 	1    1000 1450
@@
 F 0 "C17" H 3550 1550 40  0000 L CNN
 F 1 "10 uF" H 3556 1365 40  0000 L CNN
-F 2 "" H 3588 1300 30  0000 C CNN
+F 2 "Capacitors_SMD:C_0402" H 3588 1300 30  0001 C CNN
 F 3 "" H 3550 1450 60  0000 C CNN
 	1    3550 1450
@@
 F 0 "C16" H 1300 1650 40  0000 L CNN
 F 1 "0.1 uF" H 1306 1465 40  0000 L CNN
-F 2 "" H 1338 1400 30  0000 C CNN
+F 2 "Capacitors_SMD:C_0402" H 1338 1400 30  0001 C CNN
 F 3 "" H 1300 1550 60  0000 C CNN
 	1    1300 1550
@@
 F 0 "C18" H 3800 1550 40  0000 L CNN
 F 1 "10 uF" H 3806 1365 40  0000 L CNN
-F 2 "" H 3838 1300 30  0000 C CNN
+F 2 "Capacitors_SMD:C_0402" H 3838 1300 30  0001 C CNN
 F 3 "" H 3800 1450 60  0000 C CNN
 	1    3800 1450
@@
 F 0 "BT2" H 1050 4050 50  0000 C CNN
 F 1 "BATTERY" H 1050 3660 50  0000 C CNN
-F 2 "" H 1050 3850 60  0000 C CNN
+F 2 "Pin_Headers:Pin_Header_Straight_1x02" H 1050 3850 60  0001 C CNN
 F 3 "" H 1050 3850 60  0000 C CNN
 	1    1050 3850
@@
 F 0 "SW1" H 9700 3010 50  0000 C CNN
 F 1 "SW_PUSH_4" H 9550 2800 50  0000 C CNN
-F 2 "" H 9550 2900 60  0000 C CNN
+F 2 "Buttons_Switches_ThroughHole:SW_TH_Tactile_Omron_B3F-10xx" H 9550 2900 60  0001 C CNN
 F 3 "" H 9550 2900 60  0000 C CNN
 	1    9550 2900
@@
 F 0 "R21" V 10230 2900 40  0000 C CNN
 F 1 "10K" V 10157 2901 40  0000 C CNN
-F 2 "" V 10080 2900 30  0000 C CNN
+F 2 "Resistors_SMD:R_0402" V 10080 2900 30  0001 C CNN
 F 3 "" H 10150 2900 30  0000 C CNN
 	1    10150 2900
@@
 F 0 "R16" V 1980 3300 40  0000 C CNN
 F 1 "1M" V 1907 3301 40  0000 C CNN
-F 2 "" V 1830 3300 30  0000 C CNN
+F 2 "Resistors_SMD:R_0402" V 1830 3300 30  0001 C CNN
 F 3 "" H 1900 3300 30  0000 C CNN
 	1    1900 3300
@@
 F 0 "Q5" H 1150 2940 60  0000 R CNN
 F 1 "MOS_P" H 1150 2570 60  0000 R CNN
-F 2 "" H 1150 2750 60  0000 C CNN
+F 2 "TO_SOT_Packages_SMD:SOT-23_Handsoldering" H 1150 2750 60  0001 C CNN
 F 3 "" H 1150 2750 60  0000 C CNN
 	1    1150 2750
@@
 F 0 "L3" V 9450 1500 40  0000 C CNN
 F 1 "INDUCTOR" V 9600 1500 40  0000 C CNN
-F 2 "" H 9500 1500 60  0000 C CNN
+F 2 "Choke_Axial_ThroughHole:Choke_Horizontal_RM10mm" H 9500 1500 60  0001 C CNN
 F 3 "" H 9500 1500 60  0000 C CNN
 	1    9500 1500
@@
 F 0 "L4" V 9450 1750 40  0000 C CNN
 F 1 "INDUCTOR" V 9600 1750 40  0000 C CNN
-F 2 "" H 9500 1750 60  0000 C CNN
+F 2 "Choke_Axial_ThroughHole:Choke_Horizontal_RM10mm" H 9500 1750 60  0001 C CNN
 F 3 "" H 9500 1750 60  0000 C CNN
 	1    9500 1750
@@
 F 0 "R19" V 9330 5150 40  0000 C CNN
 F 1 "1M" V 9257 5151 40  0000 C CNN
-F 2 "" V 9180 5150 30  0000 C CNN
+F 2 "Resistors_SMD:R_0402" V 9180 5150 30  0001 C CNN
 F 3 "" H 9250 5150 30  0000 C CNN
 	1    9250 5150
@@
 F 0 "R20" V 9330 5750 40  0000 C CNN
 F 1 "1M" V 9257 5751 40  0000 C CNN
-F 2 "" V 9180 5750 30  0000 C CNN
+F 2 "Resistors_SMD:R_0402" V 9180 5750 30  0001 C CNN
 F 3 "" H 9250 5750 30  0000 C CNN
 	1    9250 5750
@@
 F 0 "U9" H 5750 3900 60  0000 C CNN
 F 1 "TPS63061" H 5900 3800 60  0000 C CNN
-F 2 "" H 6200 2650 60  0000 C CNN
+F 2 "Housings_SSOP:MSOP-10-1EP_3x3mm_Pitch0.5mm" H 6200 2650 60  0001 C CNN
 F 3 "" H 6200 2650 60  0000 C CNN
 	1    6050 3250
@@
 F 0 "R15" V 1980 2700 40  0000 C CNN
 F 1 "1K" V 1907 2701 40  0000 C CNN
-F 2 "" V 1830 2700 30  0000 C CNN
+F 2 "Resistors_SMD:R_0402" V 1830 2700 30  0001 C CNN
 F 3 "" H 1900 2700 30  0000 C CNN
 	1    1900 2700
@@
 F 0 "Q6" H 1150 3440 60  0000 R CNN
 F 1 "MOS_P" H 1150 3070 60  0000 R CNN
-F 2 "" H 1150 3250 60  0000 C CNN
+F 2 "TO_SOT_Packages_SMD:SOT-23_Handsoldering" H 1150 3250 60  0001 C CNN
 F 3 "" H 1150 3250 60  0000 C CNN
 	1    1150 3250
@@
 F 0 "L2" V 6950 3800 50  0000 C CNN
 F 1 "1 uH" V 7100 3800 50  0000 C CNN
-F 2 "" H 7000 3800 50  0000 C CNN
+F 2 "Inductors:IND_BOURNS_SRP1238A" H 7000 3800 50  0001 C CNN
 F 3 "" H 7000 3800 50  0000 C CNN
 	1    7000 3800
@@
 F 0 "C21" H 5325 3750 50  0000 L CNN
 F 1 "0.1 uF" H 5325 3550 50  0000 L CNN
-F 2 "" H 5338 3500 50  0000 C CNN
+F 2 "Capacitors_SMD:C_0402" H 5338 3500 50  0001 C CNN
 F 3 "" H 5300 3650 50  0000 C CNN
 	1    5300 3650
@@
 F 0 "C20" H 4425 3100 50  0000 L CNN
 F 1 "10 uF" H 4425 2900 50  0000 L CNN
-F 2 "" H 4438 2850 50  0000 C CNN
+F 2 "Capacitors_SMD:C_0402" H 4438 2850 50  0001 C CNN
 F 3 "" H 4400 3000 50  0000 C CNN
 	1    4400 3000
@@
 F 0 "C19" H 4125 3100 50  0000 L CNN
 F 1 "10 uF" H 4125 2900 50  0000 L CNN
-F 2 "" H 4138 2850 50  0000 C CNN
+F 2 "Capacitors_SMD:C_0402" H 4138 2850 50  0001 C CNN
 F 3 "" H 4100 3000 50  0000 C CNN
 	1    4100 3000
@@
 F 0 "C22" H 7125 3150 50  0000 L CNN
 F 1 "22 uF" H 7125 2950 50  0000 L CNN
-F 2 "" H 7138 2900 50  0000 C CNN
+F 2 "Capacitors_SMD:C_0402" H 7138 2900 50  0001 C CNN
 F 3 "" H 7100 3050 50  0000 C CNN
 	1    7100 3050
@@
 F 0 "C23" H 7425 3150 50  0000 L CNN
 F 1 "22 uF" H 7425 2950 50  0000 L CNN
-F 2 "" H 7438 2900 50  0000 C CNN
+F 2 "Capacitors_SMD:C_0402" H 7438 2900 50  0001 C CNN
 F 3 "" H 7400 3050 50  0000 C CNN
 	1    7400 3050
@@
 F 0 "C24" H 7725 3150 50  0000 L CNN
 F 1 "22 uF" H 7725 2950 50  0000 L CNN
-F 2 "" H 7738 2900 50  0000 C CNN
+F 2 "Capacitors_SMD:C_0402" H 7738 2900 50  0001 C CNN
 F 3 "" H 7700 3050 50  0000 C CNN
 	1    7700 3050
@@
 F 0 "BT1" H 1000 6650 50  0000 C CNN
 F 1 "BATTERY" H 1000 6260 50  0000 C CNN
-F 2 "" H 1000 6450 60  0000 C CNN
+F 2 "Pin_Headers:Pin_Header_Straight_1x02" H 1000 6450 60  0001 C CNN
 F 3 "" H 1000 6450 60  0000 C CNN
 	1    1000 6450
@@
 F 0 "Q4" H 1100 6090 60  0000 R CNN
 F 1 "MOS_P" H 1100 5720 60  0000 R CNN
-F 2 "" H 1100 5900 60  0000 C CNN
+F 2 "TO_SOT_Packages_SMD:SOT-23_Handsoldering" H 1100 5900 60  0001 C CNN
 F 3 "" H 1100 5900 60  0000 C CNN
 	1    1100 5900
@@
 F 0 "R14" V 1830 6150 50  0000 C CNN
 F 1 "1M" V 1750 6150 50  0000 C CNN
-F 2 "" V 1680 6150 50  0000 C CNN
+F 2 "Resistors_SMD:R_0402" V 1680 6150 50  0001 C CNN
 F 3 "" H 1750 6150 50  0000 C CNN
 	1    1750 6150
@@
 F 0 "D1" H 3750 5350 50  0000 C CNN
 F 1 "D_Schottky" H 3750 5150 50  0000 C CNN
-F 2 "" H 3750 5250 50  0000 C CNN
+F 2 "Diodes_SMD:MELF-RM10_Universal_Handsoldering" H 3750 5250 50  0001 C CNN
 F 3 "" H 3750 5250 50  0000 C CNN
 	1    3750 5250
@@
 F 0 "D3" H 9100 3300 50  0000 C CNN
 F 1 "DZ2J030M0L" H 9100 3100 50  0000 C CNN
-F 2 "" H 9100 3200 50  0000 C CNN
+F 2 "Diodes_SMD:MELF-RM10_Universal_Handsoldering" H 9100 3200 50  0001 C CNN
 F 3 "" H 9100 3200 50  0000 C CNN
 	1    9100 3200
@@
 F 0 "R18" V 8880 3200 50  0000 C CNN
 F 1 "100K" V 8800 3200 50  0000 C CNN
-F 2 "" V 8730 3200 50  0000 C CNN
+F 2 "Resistors_SMD:R_0402" V 8730 3200 50  0001 C CNN
 F 3 "" H 8800 3200 50  0000 C CNN
 	1    8800 3200
@@
 F 0 "D2" H 8750 2250 50  0000 C CNN
 F 1 "D_Schottky" H 8750 2050 50  0000 C CNN
-F 2 "" H 8750 2150 50  0000 C CNN
+F 2 "Diodes_SMD:MELF-RM10_Universal_Handsoldering" H 8750 2150 50  0001 C CNN
 F 3 "" H 8750 2150 50  0000 C CNN
 	1    8750 2150
@@
 F 0 "R17" V 8380 2350 50  0000 C CNN
 F 1 "100K" V 8300 2350 50  0000 C CNN
-F 2 "" V 8230 2350 50  0000 C CNN
+F 2 "Resistors_SMD:R_0402" V 8230 2350 50  0001 C CNN
 F 3 "" H 8300 2350 50  0000 C CNN
 	1    8300 2350
