File: power.sch (KiCad schematic (older format))
At the start: 33 parts, among them Q4 MOS_P, Q5 MOS_P, Q6 MOS_P, SW1 SW_PUSH_4, U8 TPS63031, U9 TPS63061

Commit message: more stuff
Parts:
- BT1: value BATTERY -> BACK BATTERY
- BT2: value BATTERY -> MAIN BATTERY
Changed lines of the file:
@@
 $EndComp
 $Comp
-L GND-RESCUE-cansatBrain #PWR045
+L GND-RESCUE-cansatBrain #PWR044
 U 1 1 5594EE74
 P 1900 1750
-F 0 "#PWR045" H 1900 1750 30  0001 C CNN
+F 0 "#PWR044" H 1900 1750 30  0001 C CNN
 F 1 "GND" H 1900 1680 30  0001 C CNN
 F 2 "" H 1900 1750 60  0000 C CNN
@@
 $EndComp
 $Comp
-L GND-RESCUE-cansatBrain #PWR046
+L GND-RESCUE-cansatBrain #PWR045
 U 1 1 5594EE7A
 P 3150 1750
-F 0 "#PWR046" H 3150 1750 30  0001 C CNN
+F 0 "#PWR045" H 3150 1750 30  0001 C CNN
 F 1 "GND" H 3150 1680 30  0001 C CNN
 F 2 "" H 3150 1750 60  0000 C CNN
@@
 $EndComp
 $Comp
-L GND-RESCUE-cansatBrain #PWR047
+L GND-RESCUE-cansatBrain #PWR046
 U 1 1 5594EE80
 P 1300 1750
-F 0 "#PWR047" H 1300 1750 30  0001 C CNN
+F 0 "#PWR046" H 1300 1750 30  0001 C CNN
 F 1 "GND" H 1300 1680 30  0001 C CNN
 F 2 "" H 1300 1750 60  0000 C CNN
@@
 $EndComp
 $Comp
-L GND-RESCUE-cansatBrain #PWR048
+L GND-RESCUE-cansatBrain #PWR047
 U 1 1 5594EE86
 P 1000 1650
-F 0 "#PWR048" H 1000 1650 30  0001 C CNN
+F 0 "#PWR047" H 1000 1650 30  0001 C CNN
 F 1 "GND" H 1000 1580 30  0001 C CNN
 F 2 "" H 1000 1650 60  0000 C CNN
@@
 $EndComp
 $Comp
-L GND-RESCUE-cansatBrain #PWR049
+L GND-RESCUE-cansatBrain #PWR048
 U 1 1 5594EE8C
 P 3550 1650
-F 0 "#PWR049" H 3550 1650 30  0001 C CNN
+F 0 "#PWR048" H 3550 1650 30  0001 C CNN
 F 1 "GND" H 3550 1580 30  0001 C CNN
 F 2 "" H 3550 1650 60  0000 C CNN
@@
 $EndComp
 $Comp
-L VCC #PWR050
+L VCC #PWR049
 U 1 1 5594EE92
 P 3550 1250
-F 0 "#PWR050" H 3550 1350 30  0001 C CNN
+F 0 "#PWR049" H 3550 1350 30  0001 C CNN
 F 1 "VCC" H 3550 1350 30  0000 C CNN
 F 2 "" H 3550 1250 60  0000 C CNN
@@
 $EndComp
 $Comp
-L GND-RESCUE-cansatBrain #PWR051
+L GND-RESCUE-cansatBrain #PWR050
 U 1 1 5594EE9F
 P 3800 1650
-F 0 "#PWR051" H 3800 1650 30  0001 C CNN
+F 0 "#PWR050" H 3800 1650 30  0001 C CNN
 F 1 "GND" H 3800 1580 30  0001 C CNN
 F 2 "" H 3800 1650 60  0000 C CNN
@@
 P 1050 3850
 F 0 "BT2" H 1050 4050 50  0000 C CNN
-F 1 "BATTERY" H 1050 3660 50  0000 C CNN
+F 1 "MAIN BATTERY" H 1050 3660 50  0000 C CNN
 F 2 "Pin_Headers:Pin_Header_Straight_1x02" H 1050 3850 60  0001 C CNN
 F 3 "" H 1050 3850 60  0000 C CNN
@@
 $EndComp
 $Comp
-L VCCA #PWR052
+L VCCA #PWR051
 U 1 1 55952BE9
 P 9850 1450
-F 0 "#PWR052" H 9850 1550 30  0001 C CNN
+F 0 "#PWR051" H 9850 1550 30  0001 C CNN
 F 1 "VCCA" H 9850 1550 30  0000 C CNN
 F 2 "" H 9850 1450 60  0000 C CNN
@@
 $EndComp
 $Comp
-L VCC #PWR053
+L VCC #PWR052
 U 1 1 55952BF6
 P 9200 1450
-F 0 "#PWR053" H 9200 1550 30  0001 C CNN
+F 0 "#PWR052" H 9200 1550 30  0001 C CNN
 F 1 "VCC" H 9200 1550 30  0000 C CNN
 F 2 "" H 9200 1450 60  0000 C CNN
@@
 $EndComp
 $Comp
-L GNDA-RESCUE-cansatBrain #PWR054
+L GNDA-RESCUE-cansatBrain #PWR053
 U 1 1 55952BFE
 P 9850 1800
-F 0 "#PWR054" H 9850 1800 40  0001 C CNN
+F 0 "#PWR053" H 9850 1800 40  0001 C CNN
 F 1 "GNDA" H 9850 1730 40  0000 C CNN
 F 2 "" H 9850 1800 60  0000 C CNN
@@
 $EndComp
 $Comp
-L GND-RESCUE-cansatBrain #PWR055
+L GND-RESCUE-cansatBrain #PWR054
 U 1 1 55952C04
 P 9200 1800
-F 0 "#PWR055" H 9200 1800 30  0001 C CNN
+F 0 "#PWR054" H 9200 1800 30  0001 C CNN
 F 1 "GND" H 9200 1730 30  0001 C CNN
 F 2 "" H 9200 1800 60  0000 C CNN
@@
 $EndComp
 $Comp
-L GND-RESCUE-cansatBrain #PWR056
+L GND-RESCUE-cansatBrain #PWR055
 U 1 1 55955FDC
 P 9250 6050
-F 0 "#PWR056" H 9250 6050 30  0001 C CNN
+F 0 "#PWR055" H 9250 6050 30  0001 C CNN
 F 1 "GND" H 9250 5980 30  0001 C CNN
 F 2 "" H 9250 6050 60  0000 C CNN
@@
 $EndComp
 $Comp
-L GND #PWR057
+L GND #PWR056
 U 1 1 56DF83C7
 P 1050 4200
-F 0 "#PWR057" H 1050 3950 50  0001 C CNN
+F 0 "#PWR056" H 1050 3950 50  0001 C CNN
 F 1 "GND" H 1050 4050 50  0000 C CNN
 F 2 "" H 1050 4200 50  0000 C CNN
@@
 $EndComp
 $Comp
-L GND #PWR058
+L GND #PWR057
 U 1 1 56DFA497
 P 1900 3550
-F 0 "#PWR058" H 1900 3300 50  0001 C CNN
+F 0 "#PWR057" H 1900 3300 50  0001 C CNN
 F 1 "GND" H 1900 3400 50  0000 C CNN
 F 2 "" H 1900 3550 50  0000 C CNN
@@
 Disconnect battery when \nUSB power is available
 $Comp
-L +5V #PWR059
+L +5V #PWR058
 U 1 1 56DFC2FC
 P 6900 2800
-F 0 "#PWR059" H 6900 2650 50  0001 C CNN
+F 0 "#PWR058" H 6900 2650 50  0001 C CNN
 F 1 "+5V" H 6900 2940 50  0000 C CNN
 F 2 "" H 6900 2800 50  0000 C CNN
@@
 $EndComp
 $Comp
-L GND #PWR060
+L GND #PWR059
 U 1 1 56DFFA3D
 P 5400 3150
-F 0 "#PWR060" H 5400 2900 50  0001 C CNN
+F 0 "#PWR059" H 5400 2900 50  0001 C CNN
 F 1 "GND" H 5400 3000 50  0000 C CNN
 F 2 "" H 5400 3150 50  0000 C CNN
@@
 $EndComp
 $Comp
-L GND #PWR061
+L GND #PWR060
 U 1 1 56E0020E
 P 5300 3800
-F 0 "#PWR061" H 5300 3550 50  0001 C CNN
+F 0 "#PWR060" H 5300 3550 50  0001 C CNN
 F 1 "GND" H 5300 3650 50  0000 C CNN
 F 2 "" H 5300 3800 50  0000 C CNN
@@
 $EndComp
 $Comp
-L GND #PWR062
+L GND #PWR061
 U 1 1 56E00B62
 P 6000 4000
-F 0 "#PWR062" H 6000 3750 50  0001 C CNN
+F 0 "#PWR061" H 6000 3750 50  0001 C CNN
 F 1 "GND" H 6000 3850 50  0000 C CNN
 F 2 "" H 6000 4000 50  0000 C CNN
@@
 $EndComp
 $Comp
-L GND #PWR063
+L GND #PWR062
 U 1 1 56E025B4
 P 7250 3200
-F 0 "#PWR063" H 7250 2950 50  0001 C CNN
+F 0 "#PWR062" H 7250 2950 50  0001 C CNN
 F 1 "GND" H 7250 3050 50  0000 C CNN
 F 2 "" H 7250 3200 50  0000 C CNN
@@
 $EndComp
 $Comp
-L GND #PWR064
+L GND #PWR063
 U 1 1 56E05829
 P 4250 3150
-F 0 "#PWR064" H 4250 2900 50  0001 C CNN
+F 0 "#PWR063" H 4250 2900 50  0001 C CNN
 F 1 "GND" H 4250 3000 50  0000 C CNN
 F 2 "" H 4250 3150 50  0000 C CNN
@@
 NoConn ~ 6600 3350
 $Comp
-L +5V #PWR065
+L +5V #PWR064
 U 1 1 56E09B9F
 P 1200 1100
-F 0 "#PWR065" H 1200 950 50  0001 C CNN
+F 0 "#PWR064" H 1200 950 50  0001 C CNN
 F 1 "+5V" H 1200 1240 50  0000 C CNN
 F 2 "" H 1200 1100 50  0000 C CNN
@@
 P 1000 6450
 F 0 "BT1" H 1000 6650 50  0000 C CNN
-F 1 "BATTERY" H 1000 6260 50  0000 C CNN
+F 1 "BACK BATTERY" H 1000 6260 50  0000 C CNN
 F 2 "Pin_Headers:Pin_Header_Straight_1x02" H 1000 6450 60  0001 C CNN
 F 3 "" H 1000 6450 60  0000 C CNN
@@
 $EndComp
 $Comp
-L GND #PWR066
+L GND #PWR065
 U 1 1 56DF79F7
 P 1000 6750
-F 0 "#PWR066" H 1000 6500 50  0001 C CNN
+F 0 "#PWR065" H 1000 6500 50  0001 C CNN
 F 1 "GND" H 1000 6600 50  0000 C CNN
 F 2 "" H 1000 6750 50  0000 C CNN
@@
 	1000 5700 1000 5550
 $Comp
-L +5V #PWR067
+L +5V #PWR066
 U 1 1 56DFA3E3
 P 1000 5550
-F 0 "#PWR067" H 1000 5400 50  0001 C CNN
+F 0 "#PWR066" H 1000 5400 50  0001 C CNN
 F 1 "+5V" H 1000 5690 50  0000 C CNN
 F 2 "" H 1000 5550 50  0000 C CNN
@@
 $EndComp
 $Comp
-L GND #PWR068
+L GND #PWR067
 U 1 1 56DFB509
 P 1750 6300
-F 0 "#PWR068" H 1750 6050 50  0001 C CNN
+F 0 "#PWR067" H 1750 6050 50  0001 C CNN
 F 1 "GND" H 1750 6150 50  0000 C CNN
 F 2 "" H 1750 6300 50  0000 C CNN
@@
 	9100 3400 9100 3550
 $Comp
-L GND #PWR069
+L GND #PWR068
 U 1 1 56E0CBC0
 P 9100 3550
-F 0 "#PWR069" H 9100 3300 50  0001 C CNN
+F 0 "#PWR068" H 9100 3300 50  0001 C CNN
 F 1 "GND" H 9100 3400 50  0000 C CNN
 F 2 "" H 9100 3550 50  0000 C CNN
@@
 	8800 3350 8800 3550
 $Comp
-L GND #PWR070
+L GND #PWR069
 U 1 1 56E05399
 P 8800 3550
-F 0 "#PWR070" H 8800 3300 50  0001 C CNN
+F 0 "#PWR069" H 8800 3300 50  0001 C CNN
 F 1 "GND" H 8800 3400 50  0000 C CNN
 F 2 "" H 8800 3550 50  0000 C CNN
@@
 $EndComp
 $Comp
-L GND #PWR071
+L GND #PWR070
 U 1 1 56E082AF
 P 8300 2500
-F 0 "#PWR071" H 8300 2250 50  0001 C CNN
+F 0 "#PWR070" H 8300 2250 50  0001 C CNN
 F 1 "GND" H 8300 2350 50  0000 C CNN
 F 2 "" H 8300 2500 50  0000 C CNN
@@
 Connection ~ 3800 1250
 $Comp
-L PWR_FLAG #FLG072
+L PWR_FLAG #FLG071
 U 1 1 56E351F7
 P 1600 2300
-F 0 "#FLG072" H 1600 2395 50  0001 C CNN
+F 0 "#FLG071" H 1600 2395 50  0001 C CNN
 F 1 "PWR_FLAG" H 1600 2480 50  0000 C CNN
 F 2 "" H 1600 2300 50  0000 C CNN
@@
 $EndComp
 $Comp
-L PWR_FLAG #FLG073
+L PWR_FLAG #FLG072
 U 1 1 56E3A3CA
 P 10200 1500
-F 0 "#FLG073" H 10200 1595 50  0001 C CNN
+F 0 "#FLG072" H 10200 1595 50  0001 C CNN
 F 1 "PWR_FLAG" H 10200 1680 50  0000 C CNN
 F 2 "" H 10200 1500 50  0000 C CNN
@@
 Connection ~ 9850 1750
 $Comp
-L PWR_FLAG #FLG074
+L PWR_FLAG #FLG073
 U 1 1 56E3A9A8
 P 10200 1750
-F 0 "#FLG074" H 10200 1845 50  0001 C CNN
+F 0 "#FLG073" H 10200 1845 50  0001 C CNN
 F 1 "PWR_FLAG" H 10200 1930 50  0000 C CNN
 F 2 "" H 10200 1750 50  0000 C CNN
@@
 	3050 1250 3800 1250
 $Comp
-L PWR_FLAG #FLG075
+L PWR_FLAG #FLG074
 U 1 1 56E3F5D8
 P 8300 1050
-F 0 "#FLG075" H 8300 1145 50  0001 C CNN
+F 0 "#FLG074" H 8300 1145 50  0001 C CNN
 F 1 "PWR_FLAG" H 8300 1230 50  0000 C CNN
 F 2 "" H 8300 1050 50  0000 C CNN
@@
 $EndComp
 $Comp
-L GND #PWR076
+L GND #PWR075
 U 1 1 56E3F630
 P 8300 1050
-F 0 "#PWR076" H 8300 800 50  0001 C CNN
+F 0 "#PWR075" H 8300 800 50  0001 C CNN
 F 1 "GND" H 8300 900 50  0000 C CNN
 F 2 "" H 8300 1050 50  0000 C CNN

Commit message: a bunch of bom stuff
Parts:
- removed C19, C20: 10 uF, Capacitors_SMD:C_0402, symbol C
- removed C21: 0.1 uF, Capacitors_SMD:C_0402, symbol C
- added C19, C20: 10uF, Capacitors_SMD:C_0805, symbol C-RESCUE-cansatBrain
- added C21: 0.1uF, Capacitors_SMD:C_0402, symbol C-RESCUE-cansatBrain
- BT1: footprint Pin_Headers:Pin_Header_Straight_1x02 -> hlib:BH13N-C; manf# (none) -> BC1/3N
- C15, C17, C18: value 10 uF -> 10uF; footprint Capacitors_SMD:C_0402 -> Capacitors_SMD:C_0805
- C16: value 0.1 uF -> 0.1uF
- C22: value 22 uF -> 22uF; footprint Capacitors_SMD:C_0402 -> Capacitors_SMD:C_0805; manf# (none) -> CL21A226MQCLQNC
- C23, C24: value 22 uF -> 22uF; footprint Capacitors_SMD:C_0402 -> Capacitors_SMD:C_0805
- D1: footprint Diodes_SMD:MELF-RM10_Universal_Handsoldering -> Diodes_SMD:SOD-123
- D2: footprint Diodes_SMD:MELF-RM10_Universal_Handsoldering -> Diodes_SMD:SOD-123; manf# (none) -> DB2W40200L
- D3: footprint Diodes_SMD:MELF-RM10_Universal_Handsoldering -> Diodes_SMD:SOD-323; manf# (none) -> DZ2J030M0L
- L1: value 1.5 uH -> 2.2uH; footprint Inductors:IND_BOURNS_SRP1238A -> Resistors_SMD:R_1210; manf# (none) -> NLCV32T-2R2M-PFR
- L2: value 1 uH -> 1uH; footprint Inductors:IND_BOURNS_SRP1238A -> hlib:SRN4026-1R0Y; manf# (none) -> SRN4026-1R0Y
- L3, L4: footprint Choke_Axial_ThroughHole:Choke_Horizontal_RM10mm -> Resistors_SMD:R_1210
- Q4, Q5, Q6: footprint TO_SOT_Packages_SMD:SOT-23_Handsoldering -> SMD:SOT-23-3
- R14: manf# (none) -> RC0402JR-071ML
- R17: manf# (none) -> CRG0402J100K/10
- R21: manf# (none) -> RC0402JR-0710KL
- SW1: footprint Buttons_Switches_ThroughHole:SW_TH_Tactile_Omron_B3F-10xx -> 1825910-4:DIP780W71L599H950Q4; manf# (none) -> 1825910-7
- U8: footprint Housings_SSOP:MSOP-10-1EP_3x3mm_Pitch0.5mm -> TPS63031:QFN10-2.5MM; manf# (none) -> TPS63031DSKR
- U9: footprint Housings_SSOP:MSOP-10-1EP_3x3mm_Pitch0.5mm -> TPS63061:WSON-10; manf# (none) -> TPS63061DSCR
Connections:
- wire segments 73 -> 76

Commit message: laid out board
Parts:
- U9: footprint TPS63061:WSON-10 -> hlib:WSON-10
Changed lines of the file:
@@
 $EndComp
 $Comp
-L GND-RESCUE-cansatBrain #PWR045
+L GND-RESCUE-cansatBrain #PWR046
 U 1 1 5594EE74
 P 1900 1750
-F 0 "#PWR045" H 1900 1750 30  0001 C CNN
+F 0 "#PWR046" H 1900 1750 30  0001 C CNN
 F 1 "GND" H 1900 1680 30  0001 C CNN
 F 2 "" H 1900 1750 60  0000 C CNN
@@
 $EndComp
 $Comp
-L GND-RESCUE-cansatBrain #PWR046
+L GND-RESCUE-cansatBrain #PWR047
 U 1 1 5594EE7A
 P 3150 1750
-F 0 "#PWR046" H 3150 1750 30  0001 C CNN
+F 0 "#PWR047" H 3150 1750 30  0001 C CNN
 F 1 "GND" H 3150 1680 30  0001 C CNN
 F 2 "" H 3150 1750 60  0000 C CNN
@@
 $EndComp
 $Comp
-L GND-RESCUE-cansatBrain #PWR047
+L GND-RESCUE-cansatBrain #PWR048
 U 1 1 5594EE80
 P 1300 1750
-F 0 "#PWR047" H 1300 1750 30  0001 C CNN
+F 0 "#PWR048" H 1300 1750 30  0001 C CNN
 F 1 "GND" H 1300 1680 30  0001 C CNN
 F 2 "" H 1300 1750 60  0000 C CNN
@@
 $EndComp
 $Comp
-L GND-RESCUE-cansatBrain #PWR048
+L GND-RESCUE-cansatBrain #PWR049
 U 1 1 5594EE86
 P 1000 1650
-F 0 "#PWR048" H 1000 1650 30  0001 C CNN
+F 0 "#PWR049" H 1000 1650 30  0001 C CNN
 F 1 "GND" H 1000 1580 30  0001 C CNN
 F 2 "" H 1000 1650 60  0000 C CNN
@@
 $EndComp
 $Comp
-L GND-RESCUE-cansatBrain #PWR049
+L GND-RESCUE-cansatBrain #PWR050
 U 1 1 5594EE8C
 P 3550 1650
-F 0 "#PWR049" H 3550 1650 30  0001 C CNN
+F 0 "#PWR050" H 3550 1650 30  0001 C CNN
 F 1 "GND" H 3550 1580 30  0001 C CNN
 F 2 "" H 3550 1650 60  0000 C CNN
@@
 $EndComp
 $Comp
-L VCC #PWR050
+L VCC #PWR051
 U 1 1 5594EE92
 P 3550 1250
-F 0 "#PWR050" H 3550 1350 30  0001 C CNN
+F 0 "#PWR051" H 3550 1350 30  0001 C CNN
 F 1 "VCC" H 3550 1350 30  0000 C CNN
 F 2 "" H 3550 1250 60  0000 C CNN
@@
 $EndComp
 $Comp
-L GND-RESCUE-cansatBrain #PWR051
+L GND-RESCUE-cansatBrain #PWR052
 U 1 1 5594EE9F
 P 3800 1650
-F 0 "#PWR051" H 3800 1650 30  0001 C CNN
+F 0 "#PWR052" H 3800 1650 30  0001 C CNN
 F 1 "GND" H 3800 1580 30  0001 C CNN
 F 2 "" H 3800 1650 60  0000 C CNN
@@
 $EndComp
 $Comp
-L VCCA #PWR052
+L VCCA #PWR053
 U 1 1 55952BE9
 P 9850 1450
-F 0 "#PWR052" H 9850 1550 30  0001 C CNN
+F 0 "#PWR053" H 9850 1550 30  0001 C CNN
 F 1 "VCCA" H 9850 1550 30  0000 C CNN
 F 2 "" H 9850 1450 60  0000 C CNN
@@
 $EndComp
 $Comp
-L VCC #PWR053
+L VCC #PWR054
 U 1 1 55952BF6
 P 9200 1450
-F 0 "#PWR053" H 9200 1550 30  0001 C CNN
+F 0 "#PWR054" H 9200 1550 30  0001 C CNN
 F 1 "VCC" H 9200 1550 30  0000 C CNN
 F 2 "" H 9200 1450 60  0000 C CNN
@@
 $EndComp
 $Comp
-L GNDA-RESCUE-cansatBrain #PWR054
+L GNDA-RESCUE-cansatBrain #PWR055
 U 1 1 55952BFE
 P 9850 1800
-F 0 "#PWR054" H 9850 1800 40  0001 C CNN
+F 0 "#PWR055" H 9850 1800 40  0001 C CNN
 F 1 "GNDA" H 9850 1730 40  0000 C CNN
 F 2 "" H 9850 1800 60  0000 C CNN
@@
 $EndComp
 $Comp
-L GND-RESCUE-cansatBrain #PWR055
+L GND-RESCUE-cansatBrain #PWR056
 U 1 1 55952C04
 P 9200 1800
-F 0 "#PWR055" H 9200 1800 30  0001 C CNN
+F 0 "#PWR056" H 9200 1800 30  0001 C CNN
 F 1 "GND" H 9200 1730 30  0001 C CNN
 F 2 "" H 9200 1800 60  0000 C CNN
@@
 $EndComp
 $Comp
-L GND-RESCUE-cansatBrain #PWR056
+L GND-RESCUE-cansatBrain #PWR057
 U 1 1 55955FDC
 P 9250 6050
-F 0 "#PWR056" H 9250 6050 30  0001 C CNN
+F 0 "#PWR057" H 9250 6050 30  0001 C CNN
 F 1 "GND" H 9250 5980 30  0001 C CNN
 F 2 "" H 9250 6050 60  0000 C CNN
@@
 F 0 "U9" H 5750 3900 60  0000 C CNN
 F 1 "TPS63061" H 5900 3800 60  0000 C CNN
-F 2 "TPS63061:WSON-10" H 6200 2650 60  0001 C CNN
+F 2 "hlib:WSON-10" H 6200 2650 60  0001 C CNN
 F 3 "" H 6200 2650 60  0000 C CNN
 F 4 "TPS63061DSCR" H 6050 3250 60  0001 C CNN "manf#"
@@
 $EndComp
 $Comp
-L GND #PWR057
+L GND #PWR058
 U 1 1 56DF83C7
 P 1050 4200
-F 0 "#PWR057" H 1050 3950 50  0001 C CNN
+F 0 "#PWR058" H 1050 3950 50  0001 C CNN
 F 1 "GND" H 1050 4050 50  0000 C CNN
 F 2 "" H 1050 4200 50  0000 C CNN
@@
 $EndComp
 $Comp
-L GND #PWR058
+L GND #PWR059
 U 1 1 56DFA497
 P 1900 3550
-F 0 "#PWR058" H 1900 3300 50  0001 C CNN
+F 0 "#PWR059" H 1900 3300 50  0001 C CNN
 F 1 "GND" H 1900 3400 50  0000 C CNN
 F 2 "" H 1900 3550 50  0000 C CNN
@@
 Disconnect battery when \nUSB power is available
 $Comp
-L +5V #PWR059
+L +5V #PWR060
 U 1 1 56DFC2FC
 P 6900 2800
-F 0 "#PWR059" H 6900 2650 50  0001 C CNN
+F 0 "#PWR060" H 6900 2650 50  0001 C CNN
 F 1 "+5V" H 6900 2940 50  0000 C CNN
 F 2 "" H 6900 2800 50  0000 C CNN
@@
 $EndComp
 $Comp
-L GND #PWR060
+L GND #PWR061
 U 1 1 56DFFA3D
 P 5400 3150
-F 0 "#PWR060" H 5400 2900 50  0001 C CNN
+F 0 "#PWR061" H 5400 2900 50  0001 C CNN
 F 1 "GND" H 5400 3000 50  0000 C CNN
 F 2 "" H 5400 3150 50  0000 C CNN
@@
 $EndComp
 $Comp
-L GND #PWR061
+L GND #PWR062
 U 1 1 56E0020E
 P 5300 3950
-F 0 "#PWR061" H 5300 3700 50  0001 C CNN
+F 0 "#PWR062" H 5300 3700 50  0001 C CNN
 F 1 "GND" H 5300 3800 50  0000 C CNN
 F 2 "" H 5300 3950 50  0000 C CNN
@@
 $EndComp
 $Comp
-L GND #PWR062
+L GND #PWR063
 U 1 1 56E00B62
 P 6000 4000
-F 0 "#PWR062" H 6000 3750 50  0001 C CNN
+F 0 "#PWR063" H 6000 3750 50  0001 C CNN
 F 1 "GND" H 6000 3850 50  0000 C CNN
 F 2 "" H 6000 4000 50  0000 C CNN
@@
 $EndComp
 $Comp
-L GND #PWR063
+L GND #PWR064
 U 1 1 56E025B4
 P 7250 3250
-F 0 "#PWR063" H 7250 3000 50  0001 C CNN
+F 0 "#PWR064" H 7250 3000 50  0001 C CNN
 F 1 "GND" H 7250 3100 50  0000 C CNN
 F 2 "" H 7250 3250 50  0000 C CNN
@@
 VIN
 $Comp
-L GND #PWR064
+L GND #PWR065
 U 1 1 56E05829
 P 4250 3350
-F 0 "#PWR064" H 4250 3100 50  0001 C CNN
+F 0 "#PWR065" H 4250 3100 50  0001 C CNN
 F 1 "GND" H 4250 3200 50  0000 C CNN
 F 2 "" H 4250 3350 50  0000 C CNN
@@
 NoConn ~ 6600 3350
 $Comp
-L +5V #PWR065
+L +5V #PWR066
 U 1 1 56E09B9F
 P 1200 1100
-F 0 "#PWR065" H 1200 950 50  0001 C CNN
+F 0 "#PWR066" H 1200 950 50  0001 C CNN
 F 1 "+5V" H 1200 1240 50  0000 C CNN
 F 2 "" H 1200 1100 50  0000 C CNN
@@
 $EndComp
 $Comp
-L GND #PWR066
+L GND #PWR067
 U 1 1 56DF79F7
 P 1000 6750
-F 0 "#PWR066" H 1000 6500 50  0001 C CNN
+F 0 "#PWR067" H 1000 6500 50  0001 C CNN
 F 1 "GND" H 1000 6600 50  0000 C CNN
 F 2 "" H 1000 6750 50  0000 C CNN
@@
 	1000 5700 1000 5550
 $Comp
-L +5V #PWR067
+L +5V #PWR068
 U 1 1 56DFA3E3
 P 1000 5550
-F 0 "#PWR067" H 1000 5400 50  0001 C CNN
+F 0 "#PWR068" H 1000 5400 50  0001 C CNN
 F 1 "+5V" H 1000 5690 50  0000 C CNN
 F 2 "" H 1000 5550 50  0000 C CNN
@@
 $EndComp
 $Comp
-L GND #PWR068
+L GND #PWR069
 U 1 1 56DFB509
 P 1750 6300
-F 0 "#PWR068" H 1750 6050 50  0001 C CNN
+F 0 "#PWR069" H 1750 6050 50  0001 C CNN
 F 1 "GND" H 1750 6150 50  0000 C CNN
 F 2 "" H 1750 6300 50  0000 C CNN
@@
 	9100 3400 9100 3550
 $Comp
-L GND #PWR069
+L GND #PWR070
 U 1 1 56E0CBC0
 P 9100 3550
-F 0 "#PWR069" H 9100 3300 50  0001 C CNN
+F 0 "#PWR070" H 9100 3300 50  0001 C CNN
 F 1 "GND" H 9100 3400 50  0000 C CNN
 F 2 "" H 9100 3550 50  0000 C CNN
@@
 	8800 3350 8800 3550
 $Comp
-L GND #PWR070
+L GND #PWR071
 U 1 1 56E05399
 P 8800 3550
-F 0 "#PWR070" H 8800 3300 50  0001 C CNN
+F 0 "#PWR071" H 8800 3300 50  0001 C CNN
 F 1 "GND" H 8800 3400 50  0000 C CNN
 F 2 "" H 8800 3550 50  0000 C CNN
@@
 $EndComp
 $Comp
-L GND #PWR071
+L GND #PWR072
 U 1 1 56E082AF
 P 8300 2500
-F 0 "#PWR071" H 8300 2250 50  0001 C CNN
+F 0 "#PWR072" H 8300 2250 50  0001 C CNN
 F 1 "GND" H 8300 2350 50  0000 C CNN
 F 2 "" H 8300 2500 50  0000 C CNN
@@
 Connection ~ 3800 1250
 $Comp
-L PWR_FLAG #FLG072
+L PWR_FLAG #FLG073
 U 1 1 56E351F7
 P 1600 2300
-F 0 "#FLG072" H 1600 2395 50  0001 C CNN
+F 0 "#FLG073" H 1600 2395 50  0001 C CNN
 F 1 "PWR_FLAG" H 1600 2480 50  0000 C CNN
 F 2 "" H 1600 2300 50  0000 C CNN
@@
 $EndComp
 $Comp
-L PWR_FLAG #FLG073
+L PWR_FLAG #FLG074
 U 1 1 56E3A3CA
 P 10200 1500
-F 0 "#FLG073" H 10200 1595 50  0001 C CNN
+F 0 "#FLG074" H 10200 1595 50  0001 C CNN
 F 1 "PWR_FLAG" H 10200 1680 50  0000 C CNN
 F 2 "" H 10200 1500 50  0000 C CNN
@@
 Connection ~ 9850 1750
 $Comp
-L PWR_FLAG #FLG074
+L PWR_FLAG #FLG075
 U 1 1 56E3A9A8
 P 10200 1750
-F 0 "#FLG074" H 10200 1845 50  0001 C CNN
+F 0 "#FLG075" H 10200 1845 50  0001 C CNN
 F 1 "PWR_FLAG" H 10200 1930 50  0000 C CNN
 F 2 "" H 10200 1750 50  0000 C CNN
@@
 	3050 1250 3800 1250
 $Comp
-L PWR_FLAG #FLG075
+L PWR_FLAG #FLG076
 U 1 1 56E3F5D8
 P 8300 1050
-F 0 "#FLG075" H 8300 1145 50  0001 C CNN
+F 0 "#FLG076" H 8300 1145 50  0001 C CNN
 F 1 "PWR_FLAG" H 8300 1230 50  0000 C CNN
 F 2 "" H 8300 1050 50  0000 C CNN
@@
 $EndComp
 $Comp
-L GND #PWR076
+L GND #PWR077
 U 1 1 56E3F630
 P 8300 1050
-F 0 "#PWR076" H 8300 800 50  0001 C CNN
+F 0 "#PWR077" H 8300 800 50  0001 C CNN
 F 1 "GND" H 8300 900 50  0000 C CNN
 F 2 "" H 8300 1050 50  0000 C CNN
