File: cansatBrain.kicad_pcb (KiCad board)
At the start: 2 copper layers, 96.5 x 99.1 mm, 74 parts, among them P11 CONN_01X03, P11 CONN_01X04, P11 I2C, Q11 MOS_P, SW11 SW_PUSH_4, U11 ArduCAM-M-2MP, U11 LS20031, U11 MPL3115A2, U11 MPU-9250, U11 TPS63031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

Commit message: stuff
Parts:
- BACKUP BT: renamed from BT11
- MAIN BT: renamed from BT11
- moved L11 88.7 mm to (177.5, 59.8)
- moved Q11 84.0 mm to (156.6, 148.3)
- moved BACKUP BT 57.9 mm to (180.9, 149.4)
- moved U11 57.9 mm to (165.0, 70.5)
- moved Q11 56.4 mm to (154.5, 70.0)
- moved C11 55.4 mm to (189.0, 56.3)
- moved Q11 48.3 mm to (183.8, 124.2)
- moved C11 47.5 mm to (185.2, 58.5)
- moved D11 45.3 mm to (162.5, 142.8)
- moved R211 43.0 mm to (131.0, 137.5)
- moved C111 43.0 mm to (195.5, 123.3)
- moved U11 42.9 mm to (184.2, 76.5)
- moved C111 38.9 mm to (192.1, 60.7)
- moved C11 38.8 mm to (185.2, 63.3)
- moved C211 36.3 mm to (143.5, 146.0)
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