File: cansatBrain.kicad_pcb (KiCad board)
At the start: 2 copper layers, 91.4 x 55.9 mm, 81 parts, among them P1 SERVO, P2 I2C, P3 PITOT, P4 SERIAL, Q1 MOS_P, Q2 MOS_P, Q3 MOS_P, Q4 MOS_P, Q5 MOS_P, Q6 MOS_P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

Commit message: ground planes
Routing:
- added copper zone on B.Cu, net GND
- added copper zone on F.Cu, net GND
- added copper zone on B.Cu, net GNDA
- added copper zone on F.Cu, net GNDA
Changed lines of the file:
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@@
+    )
+  )
+  (zone (net 6) (net_name GNDA) (layer F.Cu) (hatch edge 0.508)
+    (connect_pads (clearance 0.508))
+    (min_thickness 0.254)
+    (fill yes (arc_segments 16) (thermal_gap 0.508) (thermal_bridge_width 0.508))
+    (polygon
+      (pts
+        (xy 143.4 55.2) (xy 155.4 55.2) (xy 155.4 93.2) (xy 143.4 93.2)
+      )
+    )
+  )
+  (zone (net 2) (net_name GND) (layer F.Cu) (hatch edge 0.508)
+    (connect_pads (clearance 0.508))
+    (min_thickness 0.254)
+    (fill yes (arc_segments 16) (thermal_gap 0.508) (thermal_bridge_width 0.508))
+    (polygon
+      (pts
+        (xy 176.4 53.2) (xy 86.4 53.2) (xy 86.4 108.2) (xy 176.4 108.2)
+      )
+    )
+  )
+  (zone (net 6) (net_name GNDA) (layer B.Cu) (hatch edge 0.508)
+    (connect_pads (clearance 0.508))
+    (min_thickness 0.254)
+    (fill yes (arc_segments 16) (thermal_gap 0.508) (thermal_bridge_width 0.508))
+    (polygon
+      (pts
+        (xy 143.4 93.2) (xy 155.4 93.2) (xy 155.4 55.2) (xy 143.4 55.2)
+      )
+    )
+  )
+  (zone (net 2) (net_name GND) (layer B.Cu) (hatch edge 0.508)
+    (connect_pads (clearance 0.508))
+    (min_thickness 0.254)
+    (fill yes (arc_segments 16) (thermal_gap 0.508) (thermal_bridge_width 0.508))
+    (polygon
+      (pts
+        (xy 86.4 53.2) (xy 176.4 53.2) (xy 176.4 108.2) (xy 86.4 108.2)
+      )
     )
   )
