File: cansatBrain.sch (KiCad schematic (older format))
At the start: 41 parts, among them P1 SERVO, P2 I2C, P3 PITOT, P4 SERIAL, Q1 MOS_P, Q2 MOS_P, Q3 MOS_P, U1 Teensy_LC, U2 MPL3115A2, U3 microSD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

Commit message: a bunch of bom stuff
Parts:
- added R22, R23: 1K, Resistors_SMD:R_0402, symbol R-RESCUE-cansatBrain
- added R24, R25: 10k, Resistors_SMD:R_0402, symbol R
- C1, C5: footprint Capacitors_SMD:C_0402 -> Capacitors_SMD:C_0805; manf# (none) -> C0805C106Z8VACTU
- C10, C13, C14: footprint Capacitors_SMD:C_0402 -> Capacitors_SMD:C_0805
- C2, C3: manf# (none) -> CL05A104KP5NNNC
- C4: manf# (none) -> 04026D105KAT2A
- C6: manf# (none) -> CC0402KRX7R8BB103
- Q1: footprint TO_SOT_Packages_SMD:SOT-23_Handsoldering -> SMD:SOT-23-3; manf# (none) -> PMV48XP,215
- Q2, Q3: footprint TO_SOT_Packages_SMD:SOT-23_Handsoldering -> SMD:SOT-23-3
- R1: manf# (none) -> CRG0402J100R/10
- R2: manf# (none) -> RC0402JR-071ML
- R3: manf# (none) -> RC0402JR-071KL
- U1: footprint Housings_DIP:DIP-28_W15.24mm -> hlib:Teensy_3.1
- U2: footprint SMD_Packages:SOIC-8-N -> MPL3115A2:LGA8
- U3: footprint Pin_Headers:Pin_Header_Straight_1x06 -> DM3CS-SF:HRS_DM3CS-SF; manf# (none) -> DM3CS-SF
- U4: footprint Housings_DFN_QFN:QFN-24-1EP_3x3mm_Pitch0.4mm -> MPU-9250:QFN-24%2f3MM
- U6: footprint Housings_DIP:DIP-20_W7.62mm_LongPads -> XB24-Z7WIT-004:DIP-20
Connections:
- net SCL: now also R25.2
- net SDA: now also R24.2
- net VCC: now also R24.1, R25.1
- net XTRA_RX: now also R22.1; no longer U1.0 (0(RX1))
- net XTRA_TX: now also R23.1; no longer U1.1 (1(TX1))
- new net: R22.2, U1.0 (0(RX1))
- new net: R23.2, U1.1 (1(TX1))
Other:
- moved on the sheet: P3, Q3, R10, R11, R12, R13

Commit message: laid out board
Parts:
- added Q7: MOS_P, SMD:SOT-23-3, symbol MOS_P
- added R26: 100, Resistors_SMD:R_0402, symbol R-RESCUE-cansatBrain
- added R27: 1M, Resistors_SMD:R_0402, symbol R-RESCUE-cansatBrain
- U3: footprint DM3CS-SF:HRS_DM3CS-SF -> hlib:HRS_DM3CS-SF
- U4: footprint MPU-9250:QFN-24%2f3MM -> hlib:QFN-24_3x3MM; manf# (none) -> MPU-9250
- U6: footprint XB24-Z7WIT-004:DIP-20 -> hlib:xbee
Connections:
- net +5V: no longer U7.6 (+5V)
- net GND: now also R27.1
- net VCC: now also U7.6 (+5V), Q7.2 (S); no longer C1.1, U1.26 (Vin), U4.1 (RESV)
- net VCCA: now also U4.1 (RESV)
- net VUSB: now also U1.26 (Vin), R26.2; no longer U1.~ (VUSB)
- net SD_POWER: now reaches C10.1, C7.1, C9.1, Q2.3 (D), U3.4 (VDD)
- net TEENSY_POWER: now reaches U1.24 (3.3V)
- net TEENSY_POWER: now also C1.1, Q7.3 (D)
- net SERVO_POWER: now reaches P1.2 (P2), Q1.3 (D)
- net PITOT_POWER: now reaches P3.2 (P2), Q3.3 (D)
- new net: Q7.1 (G), R26.1, R27.2
Other:
- moved on the sheet: C1
Changed lines of the file:
@@
 F 0 "U4" H 5350 2350 60  0000 C CNN
 F 1 "MPU-9250" H 5350 950 60  0000 C CNN
-F 2 "MPU-9250:QFN-24%2f3MM" H 5450 1750 60  0001 C CNN
+F 2 "hlib:QFN-24_3x3MM" H 5450 1750 60  0001 C CNN
 F 3 "" H 5450 1750 60  0000 C CNN
+F 4 "MPU-9250" H 5350 1650 60  0001 C CNN "manf#"
 	1    5350 1650
 	1    0    0    -1
@@
 F 0 "U6" H 7950 2400 60  0000 C CNN
 F 1 "XBee" H 8000 800 60  0000 C CNN
-F 2 "XB24-Z7WIT-004:DIP-20" H 9350 1050 60  0001 C CNN
+F 2 "hlib:xbee" H 9350 1050 60  0001 C CNN
 F 3 "" H 9350 1050 60  0000 C CNN
 	1    8650 1600
@@
 F 0 "U3" H 5000 7100 60  0000 C CNN
 F 1 "microSD" H 5050 6500 60  0000 C CNN
-F 2 "DM3CS-SF:HRS_DM3CS-SF" H 4950 6750 60  0001 C CNN
+F 2 "hlib:HRS_DM3CS-SF" H 4950 6750 60  0001 C CNN
 F 3 "" H 4950 6750 60  0000 C CNN
 F 4 "DM3CS-SF" H 5250 6800 60  0001 C CNN "manf#"
@@
 L VCC #PWR02
 U 1 1 55912D5A
-P 900 4000
-F 0 "#PWR02" H 900 4100 30  0001 C CNN
-F 1 "VCC" H 900 4100 30  0000 C CNN
-F 2 "" H 900 4000 60  0000 C CNN
-F 3 "" H 900 4000 60  0000 C CNN
-	1    900  4000
-	1    0    0    -1
-$EndComp
-NoConn ~ 1050 4150
+P 700 5200
+F 0 "#PWR02" H 700 5300 30  0001 C CNN
+F 1 "VCC" H 700 5300 30  0000 C CNN
+F 2 "" H 700 5200 60  0000 C CNN
+F 3 "" H 700 5200 60  0000 C CNN
+	1    700  5200
+	1    0    0    -1
+$EndComp
 Text Label 2850 5550 0    60   ~ 0
 SDA
@@
 	1050 7400 850  7400
 Connection ~ 850  7400
-Wire Wire Line
-	1050 3850 550  3850
-Wire Wire Line
-	900  4000 900  4050
-Wire Wire Line
-	700  4050 1050 4050
 Wire Wire Line
 	2500 5550 2850 5550
@@
 Wire Wire Line
 	4250 1700 4750 1700
-$Comp
-L VCC #PWR027
-U 1 1 55970828
-P 6050 1650
-F 0 "#PWR027" H 6050 1750 30  0001 C CNN
-F 1 "VCC" H 6050 1750 30  0000 C CNN
-F 2 "" H 6050 1650 60  0000 C CNN
-F 3 "" H 6050 1650 60  0000 C CNN
-	1    6050 1650
-	1    0    0    -1
-$EndComp
 Wire Wire Line
 	6050 1650 6050 1700
@@
 NoConn ~ 5950 1800
 $Comp
-L GNDA-RESCUE-cansatBrain #PWR028
+L GNDA-RESCUE-cansatBrain #PWR027
 U 1 1 5597096F
 P 6000 1950
-F 0 "#PWR028" H 6000 1950 40  0001 C CNN
+F 0 "#PWR027" H 6000 1950 40  0001 C CNN
 F 1 "GNDA" H 6000 1880 40  0000 C CNN
 F 2 "" H 6000 1950 60  0000 C CNN
@@
 NoConn ~ 5950 1400
 $Comp
-L GNDA-RESCUE-cansatBrain #PWR029
+L GNDA-RESCUE-cansatBrain #PWR028
 U 1 1 55970FAD
 P 4300 1150
-F 0 "#PWR029" H 4300 1150 40  0001 C CNN
+F 0 "#PWR028" H 4300 1150 40  0001 C CNN
 F 1 "GNDA" H 4300 1080 40  0000 C CNN
 F 2 "" H 4300 1150 60  0000 C CNN
@@
 $EndComp
 $Comp
-L GNDA-RESCUE-cansatBrain #PWR030
+L GNDA-RESCUE-cansatBrain #PWR029
 U 1 1 5597609C
 P 4350 2550
-F 0 "#PWR030" H 4350 2550 40  0001 C CNN
+F 0 "#PWR029" H 4350 2550 40  0001 C CNN
 F 1 "GNDA" H 4350 2480 40  0000 C CNN
 F 2 "" H 4350 2550 60  0000 C CNN
@@
 $EndComp
 $Comp
-L GNDA-RESCUE-cansatBrain #PWR031
+L GNDA-RESCUE-cansatBrain #PWR030
 U 1 1 559760A2
 P 4100 2550
-F 0 "#PWR031" H 4100 2550 40  0001 C CNN
+F 0 "#PWR030" H 4100 2550 40  0001 C CNN
 F 1 "GNDA" H 4100 2480 40  0000 C CNN
 F 2 "" H 4100 2550 60  0000 C CNN
@@
 $EndComp
 $Comp
-L GNDA-RESCUE-cansatBrain #PWR032
+L GNDA-RESCUE-cansatBrain #PWR031
 U 1 1 559760A8
 P 3850 2550
-F 0 "#PWR032" H 3850 2550 40  0001 C CNN
+F 0 "#PWR031" H 3850 2550 40  0001 C CNN
 F 1 "GNDA" H 3850 2480 40  0000 C CNN
 F 2 "" H 3850 2550 60  0000 C CNN
@@
 L C-RESCUE-cansatBrain C1
 U 1 1 5598A4C3
-P 700 4250
-F 0 "C1" H 700 4350 40  0000 L CNN
-F 1 "10uF" H 706 4165 40  0000 L CNN
-F 2 "Capacitors_SMD:C_0805" H 738 4100 30  0001 C CNN
-F 3 "" H 700 4250 60  0000 C CNN
-F 4 "C0805C106Z8VACTU" H 700 4250 60  0001 C CNN "manf#"
-	1    700  4250
+P 1000 4400
+F 0 "C1" H 1000 4500 40  0000 L CNN
+F 1 "10uF" H 1006 4315 40  0000 L CNN
+F 2 "Capacitors_SMD:C_0805" H 1038 4250 30  0001 C CNN
+F 3 "" H 1000 4400 60  0000 C CNN
+F 4 "C0805C106Z8VACTU" H 1000 4400 60  0001 C CNN "manf#"
+	1    1000 4400
+	1    0    0    -1
+$EndComp
+$Comp
+L GND-RESCUE-cansatBrain #PWR032
+U 1 1 5598A51D
+P 1000 4600
+F 0 "#PWR032" H 1000 4600 30  0001 C CNN
+F 1 "GND" H 1000 4530 30  0001 C CNN
+F 2 "" H 1000 4600 60  0000 C CNN
+F 3 "" H 1000 4600 60  0000 C CNN
+	1    1000 4600
 	1    0    0    -1
 $EndComp
 $Comp
 L GND-RESCUE-cansatBrain #PWR033
-U 1 1 5598A51D
-P 700 4450
-F 0 "#PWR033" H 700 4450 30  0001 C CNN
-F 1 "GND" H 700 4380 30  0001 C CNN
-F 2 "" H 700 4450 60  0000 C CNN
-F 3 "" H 700 4450 60  0000 C CNN
-	1    700  4450
-	1    0    0    -1
-$EndComp
-Connection ~ 900  4050
-$Comp
-L GND-RESCUE-cansatBrain #PWR034
 U 1 1 5598DC65
 P 6850 1350
-F 0 "#PWR034" H 6850 1350 30  0001 C CNN
+F 0 "#PWR033" H 6850 1350 30  0001 C CNN
 F 1 "GND" H 6850 1280 30  0001 C CNN
 F 2 "" H 6850 1350 60  0000 C CNN
@@
 Wire Wire Line
 	8950 3250 8950 3100
-$Comp
-L +5V #PWR035
-U 1 1 56E1A199
-P 8950 3100
-F 0 "#PWR035" H 8950 2950 50  0001 C CNN
-F 1 "+5V" H 8950 3240 50  0000 C CNN
-F 2 "" H 8950 3100 50  0000 C CNN
-F 3 "" H 8950 3100 50  0000 C CNN
-	1    8950 3100
-	1    0    0    -1
-$EndComp
 Wire Wire Line
 	9300 3450 8950 3450
@@
 	8950 4100 9300 4100
 $Comp
-L GND #PWR036
+L GND #PWR034
 U 1 1 56E1D429
 P 9800 4400
-F 0 "#PWR036" H 9800 4150 50  0001 C CNN
+F 0 "#PWR034" H 9800 4150 50  0001 C CNN
 F 1 "GND" H 9800 4250 50  0000 C CNN
 F 2 "" H 9800 4400 50  0000 C CNN
@@
 	8600 6100 8600 6250
 $Comp
-L GND #PWR037
+L GND #PWR035
 U 1 1 56E22EFE
 P 8600 6250
-F 0 "#PWR037" H 8600 6000 50  0001 C CNN
+F 0 "#PWR035" H 8600 6000 50  0001 C CNN
 F 1 "GND" H 8600 6100 50  0000 C CNN
 F 2 "" H 8600 6250 50  0000 C CNN
@@
 $EndComp
 $Comp
-L VCC #PWR038
+L VCC #PWR036
 U 1 1 56E26A49
 P 8450 6450
-F 0 "#PWR038" H 8450 6550 30  0001 C CNN
+F 0 "#PWR036" H 8450 6550 30  0001 C CNN
 F 1 "VCC" H 8450 6550 30  0000 C CNN
 F 2 "" H 8450 6450 60  0000 C CNN
@@
 	6750 6450 7250 6450
 $Comp
-L +5V #PWR039
+L +5V #PWR037
 U 1 1 56E2B802
 P 7700 5900
-F 0 "#PWR039" H 7700 5750 50  0001 C CNN
+F 0 "#PWR037" H 7700 5750 50  0001 C CNN
 F 1 "+5V" H 7700 6040 50  0000 C CNN
 F 2 "" H 7700 5900 50  0000 C CNN
@@
 $EndComp
 $Comp
-L GND #PWR040
+L GND #PWR038
 U 1 1 56E2EB19
 P 9400 6200
-F 0 "#PWR040" H 9400 5950 50  0001 C CNN
+F 0 "#PWR038" H 9400 5950 50  0001 C CNN
 F 1 "GND" H 9400 6050 50  0000 C CNN
 F 2 "" H 9400 6200 50  0000 C CNN
@@
 MOSI
 $Comp
-L PWR_FLAG #FLG041
+L PWR_FLAG #FLG039
 U 1 1 56E4921F
 P 5700 6200
-F 0 "#FLG041" H 5700 6295 50  0001 C CNN
+F 0 "#FLG039" H 5700 6295 50  0001 C CNN
 F 1 "PWR_FLAG" H 5700 6380 50  0000 C CNN
 F 2 "" H 5700 6200 50  0000 C CNN
@@
 XTRA_RX
 $Comp
-L VCC #PWR042
+L VCC #PWR040
 U 1 1 56E4B58A
 P 6300 5000
-F 0 "#PWR042" H 6300 4850 50  0001 C CNN
+F 0 "#PWR040" H 6300 4850 50  0001 C CNN
 F 1 "VCC" H 6300 5150 50  0000 C CNN
 F 2 "" H 6300 5000 50  0000 C CNN
@@
 $EndComp
 $Comp
-L GND #PWR043
+L GND #PWR041
 U 1 1 56E4B6EB
 P 6300 5150
-F 0 "#PWR043" H 6300 4900 50  0001 C CNN
+F 0 "#PWR041" H 6300 4900 50  0001 C CNN
 F 1 "GND" H 6300 5000 50  0000 C CNN
 F 2 "" H 6300 5150 50  0000 C CNN
@@
 	3000 3850 3350 3850
 $Comp
-L VCC #PWR044
+L VCC #PWR042
 U 1 1 56F293BC
 P 7850 4450
-F 0 "#PWR044" H 7850 4300 50  0001 C CNN
+F 0 "#PWR042" H 7850 4300 50  0001 C CNN
 F 1 "VCC" H 7850 4600 50  0000 C CNN
 F 2 "" H 7850 4450 50  0000 C CNN
@@
 $EndComp
 Wire Wire Line
-	8050 4500 7650 4500
+	7650 4500 8050 4500
 Wire Wire Line
 	7850 4450 7850 4500
@@
 Text Label 8050 5000 0    60   ~ 0
 SCL
+$Comp
+L MOS_P Q7
+U 1 1 56F38971
+P 700 4800
+F 0 "Q7" H 700 4990 60  0000 R CNN
+F 1 "MOS_P" H 700 4620 60  0000 R CNN
+F 2 "SMD:SOT-23-3" H 700 4800 60  0001 C CNN
+F 3 "" H 700 4800 60  0000 C CNN
+F 4 "PMV48XP,215" H 700 4800 60  0001 C CNN "manf#"
+	1    700  4800
+	-1   0    0    -1
+$EndComp
+Wire Wire Line
+	600  4600 600  4150
+Wire Wire Line
+	600  4150 1050 4150
+Wire Wire Line
+	1000 4200 1000 4150
+Connection ~ 1000 4150
+Wire Wire Line
+	600  5000 600  5200
+Wire Wire Line
+	600  5200 700  5200
+$Comp
+L R-RESCUE-cansatBrain R27
+U 1 1 56F43E76
+P 1100 5900
+F 0 "R27" V 1180 5900 40  0000 C CNN
+F 1 "1M" V 1107 5901 40  0000 C CNN
+F 2 "Resistors_SMD:R_0402" V 1030 5900 30  0001 C CNN
+F 3 "" H 1100 5900 30  0000 C CNN
+F 4 "RC0402JR-071ML" H 1100 5900 60  0001 C CNN "manf#"
+	1    1100 5900
+	-1   0    0    1
+$EndComp
+Wire Wire Line
+	1100 4800 1100 5650
+Wire Wire Line
+	1100 4800 900  4800
+$Comp
+L GND #PWR043
+U 1 1 56F45046
+P 1100 6150
+F 0 "#PWR043" H 1100 5900 50  0001 C CNN
+F 1 "GND" H 1100 6000 50  0000 C CNN
+F 2 "" H 1100 6150 50  0000 C CNN
+F 3 "" H 1100 6150 50  0000 C CNN
+	1    1100 6150
+	1    0    0    -1
+$EndComp
+Wire Wire Line
+	550  3850 800  3850
+Wire Wire Line
+	800  3850 800  4050
+Wire Wire Line
+	800  4050 1050 4050
+NoConn ~ 1050 3850
+$Comp
+L R-RESCUE-cansatBrain R26
+U 1 1 56F483A7
+P 800 5550
+F 0 "R26" V 880 5550 40  0000 C CNN
+F 1 "100" V 807 5551 40  0000 C CNN
+F 2 "Resistors_SMD:R_0402" V 730 5550 30  0001 C CNN
+F 3 "" H 800 5550 30  0000 C CNN
+F 4 "CRG0402J100R/10" H 800 5550 60  0001 C CNN "manf#"
+	1    800  5550
+	0    1    1    0
+$EndComp
+Wire Wire Line
+	1050 5550 1100 5550
+Connection ~ 1100 5550
+Wire Wire Line
+	550  5550 550  5900
+Text Label 550  5900 0    60   ~ 0
+VUSB
+Text Label 5950 6300 0    60   ~ 0
+SD_POWER
+Text Label 2350 1100 0    60   ~ 0
+SERVO_POWER
+Text Label 8200 6000 0    60   ~ 0
+PITOT_POWER
+Text Label 600  4400 0    60   ~ 0
+TEENSY_POWER
+$Comp
+L VCCA #PWR044
+U 1 1 56F310E7
+P 6050 1650
+F 0 "#PWR044" H 6050 1750 30  0001 C CNN
+F 1 "VCCA" H 6050 1750 30  0000 C CNN
+F 2 "" H 6050 1650 60  0000 C CNN
+F 3 "" H 6050 1650 60  0000 C CNN
+	1    6050 1650
+	1    0    0    -1
+$EndComp
+$Comp
+L VCC #PWR045
+U 1 1 56F3B0AF
+P 8950 3100
+F 0 "#PWR045" H 8950 2950 50  0001 C CNN
+F 1 "VCC" H 8950 3250 50  0000 C CNN
+F 2 "" H 8950 3100 50  0000 C CNN
+F 3 "" H 8950 3100 50  0000 C CNN
+	1    8950 3100
+	1    0    0    -1
+$EndComp
 $EndSCHEMATC
